File: power.kicad_sch (KiCad schematic)
At the start: 77 parts, among them U1 TLV74018PDBVR, U14 TMI3411, U17 TMI3408F, U3 MP9943GQ-Z, U7 TMI3113B

Commit message: 22_09_26_23_16
Parts:
- removed RST1: (no value), TestPoint:TestPoint_Pad_D1.0mm, symbol ProPrj_Ope-easyedapro:Test-Point
Connections:
- no-connect marks 1 -> 2
Other:
- note added: "short to gnd for reset"
Changed lines of the file:
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@@
 		)
 	)
+	(text "short to gnd for reset"
+		(exclude_from_sim no)
+		(at 140.208 60.706 0)
+		(effects
+			(font
+				(size 1.27 1.27)
+			)
+		)
+	)
 	(junction
 		(at 39.37 30.48)
@@
 	)
 	(no_connect
+		(at 140.97 58.42)
+	)
+	(no_connect
 		(at 134.62 163.83)
 	)
@@
 					(unit 1)
 				)
-			)
-		)
-	)
-	(symbol
-		(lib_id "ProPrj_Ope-easyedapro:Test-Point")
-		(at 140.97 58.42 180)
-		(unit 1)
-		(body_style 1)
-		(exclude_from_sim no)
-		(in_bom no)
-		(on_board yes)
-		(in_pos_files yes)
-		(dnp no)
-		(property "Reference" "RST1"
-			(at 145.288 58.928 0)
-			(hide yes)
-			(show_name no)
-			(do_not_autoplace no)
-			(effects
-				(font
-					(size 1.2446 1.2446)
-				)
-				(justify left bottom)
-			)
-		)
-		(property "Value" ""
-			(at 140.97 58.42 0)
-			(show_name no)
-			(do_not_autoplace no)
-			(effects
-				(font
-					(size 1.27 1.27)
-				)
-			)
-		)
-		(property "Footprint" "TestPoint:TestPoint_Pad_D1.0mm"
-			(at 140.97 58.42 0)
-			(hide yes)
-			(show_name no)
-			(do_not_autoplace no)
-			(effects
-				(font
-					(size 1.27 1.27)
-				)
-			)
-		)
-		(property "Datasheet" ""
-			(at 140.97 58.42 0)
-			(hide yes)
-			(show_name no)
-			(do_not_autoplace no)
-			(effects
-				(font
-					(size 1.27 1.27)
-				)
-			)
-		)
-		(property "Description" ""
-			(at 140.97 58.42 0)
-			(hide yes)
-			(show_name no)
-			(do_not_autoplace no)
-			(effects
-				(font
-					(size 1.27 1.27)
-				)
-			)
-		)
-		(pin "1"
-		)
-		(instances
-			(project "ssq338q_V1"
-				(path "/f9b84c53-a818-495f-9733-64f8168cff99/cec0b6a4-c0a0-489c-9f3c-cf508f35c098"
-					(reference "RST1")
-					(unit 1)
-				)

Commit message: minor changes and prepared BOM
Parts:
- C149, C152, C154, C155, C157, C158, C160, C161, C162, C166, C167, C168, C169, C170, C171, C172, C173, C174, C175, C176, C63, C70, C71, C72, C88: LCSC Part Name 100nF ±10% 50V -> (none)
- C33, C35: LCSC Part Name 10uF ±20% 25V -> (none)
- R15, R23: value 100K -> 100k
- R36: value 75K -> 75k
- R37: value 15K -> 15k
- R38: value 10K -> 10k
Changed lines of the file:
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@@
 			)
 		)
-		(property "LCSC Part Name" "100nF ±10% 50V"
+		(property "LCSC Part Name" ""
 			(at 39.37 129.54 0)
 			(hide yes)
@@
 			)
 		)
-		(property "LCSC Part Name" "100nF ±10% 50V"
+		(property "LCSC Part Name" ""
 			(at 238.76 31.75 0)
 			(hide yes)
@@
 			)
 		)
-		(property "Value" "100K"
+		(property "Value" "100k"
 			(at 27.94 131.572 90)
 			(show_name no)
@@
 			)
 		)
-		(property "LCSC Part Name" "100nF ±10% 50V"
+		(property "LCSC Part Name" ""
 			(at 261.62 31.75 0)
 			(hide yes)
@@
 			)
 		)
-		(property "Value" "10K"
+		(property "Value" "10k"
 			(at 72.39 172.72 90)
 			(show_name no)
@@
 			)
 		)
-		(property "LCSC Part Name" "100nF ±10% 50V"
+		(property "LCSC Part Name" ""
 			(at 223.52 78.74 0)
 			(hide yes)
@@
 			)
 		)
-		(property "LCSC Part Name" "100nF ±10% 50V"
+		(property "LCSC Part Name" ""
 			(at 261.62 78.74 0)
 			(hide yes)
@@
 			)
 		)
-		(property "LCSC Part Name" "100nF ±10% 50V"
+		(property "LCSC Part Name" ""
 			(at 29.21 115.57 0)
 			(hide yes)
@@
 			)
 		)
-		(property "LCSC Part Name" "100nF ±10% 50V"
+		(property "LCSC Part Name" ""
 			(at 43.18 88.9 0)
 			(hide yes)
@@
 			)
 		)
-		(property "LCSC Part Name" "100nF ±10% 50V"
+		(property "LCSC Part Name" ""
 			(at 276.86 78.74 0)
 			(hide yes)
@@
 			)
 		)
-		(property "Value" "15K"
+		(property "Value" "15k"
 			(at 72.39 160.02 90)
 			(show_name no)
@@
 			)
 		)
-		(property "LCSC Part Name" "100nF ±10% 50V"
+		(property "LCSC Part Name" ""
 			(at 215.9 31.75 0)
 			(hide yes)
@@
 			)
 		)
-		(property "LCSC Part Name" "100nF ±10% 50V"
+		(property "LCSC Part Name" ""
 			(at 215.9 78.74 0)
 			(hide yes)
@@
 			)
 		)
-		(property "LCSC Part Name" "100nF ±10% 50V"
+		(property "LCSC Part Name" ""
 			(at 208.28 55.88 0)
 			(hide yes)
@@
 			)
 		)
-		(property "LCSC Part Name" "10uF ±20% 25V"
+		(property "LCSC Part Name" ""
 			(at 140.97 163.83 0)
 			(hide yes)
@@
 			)
 		)
-		(property "LCSC Part Name" "100nF ±10% 50V"
+		(property "LCSC Part Name" ""
 			(at 29.21 162.56 0)
 			(hide yes)
@@
 			)
 		)
-		(property "LCSC Part Name" "100nF ±10% 50V"
+		(property "LCSC Part Name" ""
 			(at 231.14 78.74 0)
 			(hide yes)
@@
 			)
 		)
-		(property "LCSC Part Name" "100nF ±10% 50V"
+		(property "LCSC Part Name" ""
 			(at 193.04 55.88 0)
 			(hide yes)
@@
 			)
 		)
-		(property "LCSC Part Name" "100nF ±10% 50V"
+		(property "LCSC Part Name" ""
 			(at 200.66 55.88 0)
 			(hide yes)
@@
 			)
 		)
-		(property "LCSC Part Name" "100nF ±10% 50V"
+		(property "LCSC Part Name" ""
 			(at 208.28 78.74 0)
 			(hide yes)
@@
 			)
 		)
-		(property "LCSC Part Name" "100nF ±10% 50V"
+		(property "LCSC Part Name" ""
 			(at 254 31.75 0)
 			(hide yes)
@@
 			)
 		)
-		(property "LCSC Part Name" "100nF ±10% 50V"
+		(property "LCSC Part Name" ""
 			(at 246.38 78.74 0)
 			(hide yes)
@@
 			)
 		)
-		(property "LCSC Part Name" "100nF ±10% 50V"
+		(property "LCSC Part Name" ""
 			(at 254 78.74 0)
 			(hide yes)
@@
 			)
 		)
-		(property "LCSC Part Name" "100nF ±10% 50V"
+		(property "LCSC Part Name" ""
 			(at 246.38 31.75 0)
 			(hide yes)
@@
 			)
 		)
-		(property "LCSC Part Name" "100nF ±10% 50V"
+		(property "LCSC Part Name" ""
 			(at 215.9 55.88 0)
 			(hide yes)
@@
 			)
 		)
-		(property "LCSC Part Name" "10uF ±20% 25V"
+		(property "LCSC Part Name" ""
 			(at 106.68 163.83 0)
 			(hide yes)
@@
 			)
 		)
-		(property "LCSC Part Name" "100nF ±10% 50V"
+		(property "LCSC Part Name" ""
 			(at 231.14 31.75 0)
 			(hide yes)
@@
 			)
 		)
-		(property "LCSC Part Name" "100nF ±10% 50V"
+		(property "LCSC Part Name" ""
 			(at 269.24 78.74 0)
 			(hide yes)
@@
 			)
 		)
-		(property "LCSC Part Name" "100nF ±10% 50V"
+		(property "LCSC Part Name" ""
 			(at 238.76 78.74 0)
 			(hide yes)
@@
 			)
 		)
-		(property "LCSC Part Name" "100nF ±10% 50V"
+		(property "LCSC Part Name" ""
 			(at 40.64 171.45 0)
 			(hide yes)
@@
 			)
 		)
-		(property "Value" "75K"
+		(property "Value" "75k"
 			(at 72.39 128.27 90)
 			(show_name no)
@@
 			)
 		)
-		(property "Value" "100K"
+		(property "Value" "100k"
 			(at 29.464 91.694 90)
 			(show_name no)
